File: kicad/iobus2.sch (KiCad schematic (older format))
At the start: 18 parts, among them J18 Conn_01x38_Male, SW2 SW_DIP-8-SMT-HALFSIZE, U20 PCA9685, U21 MCP4728, U22 MCP4728, U23 MCP4728, U24 MCP4728

Commit message: a msg
Parts:
- C53, C57, C58, C59, C64: value 100nF -> 100 nF
- R38, R39, R40, R57, R58, R59: value 10k -> 10 k
Changed lines of the file:
@@
 EESchema Schematic File Version 4
 LIBS:ass_shield-cache
-EELAYER 26 0
+EELAYER 29 0
 EELAYER END
 $Descr A4 11693 8268
@@
 P 4900 2650
 F 0 "R38" V 4693 2650 50  0000 C CNN
-F 1 "10k" V 4784 2650 50  0000 C CNN
+F 1 "10 k" V 4784 2650 50  0000 C CNN
 F 2 "Resistor_SMD:R_0402_1005Metric" V 4800 2700 50  0001 C CNN
 F 3 "" H 4900 2750 50  0001 C CNN
@@
 P 4900 2750
 F 0 "R39" V 4693 2750 50  0000 C CNN
-F 1 "10k" V 4784 2750 50  0000 C CNN
+F 1 "10 k" V 4784 2750 50  0000 C CNN
 F 2 "Resistor_SMD:R_0402_1005Metric" V 4800 2800 50  0001 C CNN
 F 3 "" H 4900 2850 50  0001 C CNN
@@
 P 4900 2850
 F 0 "R40" V 4693 2850 50  0000 C CNN
-F 1 "10k" V 4784 2850 50  0000 C CNN
+F 1 "10 k" V 4784 2850 50  0000 C CNN
 F 2 "Resistor_SMD:R_0402_1005Metric" V 4800 2900 50  0001 C CNN
 F 3 "" H 4900 2950 50  0001 C CNN
@@
 P 4900 2950
 F 0 "R57" V 4693 2950 50  0000 C CNN
-F 1 "10k" V 4784 2950 50  0000 C CNN
+F 1 "10 k" V 4784 2950 50  0000 C CNN
 F 2 "Resistor_SMD:R_0402_1005Metric" V 4800 3000 50  0001 C CNN
 F 3 "" H 4900 3050 50  0001 C CNN
@@
 P 4900 3050
 F 0 "R58" V 4693 3050 50  0000 C CNN
-F 1 "10k" V 4784 3050 50  0000 C CNN
+F 1 "10 k" V 4784 3050 50  0000 C CNN
 F 2 "Resistor_SMD:R_0402_1005Metric" V 4800 3100 50  0001 C CNN
 F 3 "" H 4900 3150 50  0001 C CNN
@@
 P 800 2650
 F 0 "R59" V 593 2650 50  0000 C CNN
-F 1 "10k" V 684 2650 50  0000 C CNN
+F 1 "10 k" V 684 2650 50  0000 C CNN
 F 2 "Resistor_SMD:R_0402_1005Metric" V 700 2700 50  0001 C CNN
 F 3 "" H 800 2750 50  0001 C CNN
@@
 P 1850 3650
 F 0 "C53" V 1598 3650 50  0000 C CNN
-F 1 "100nF" V 1689 3650 50  0000 C CNN
+F 1 "100 nF" V 1689 3650 50  0000 C CNN
 F 2 "Capacitor_SMD:C_0402_1005Metric" V 1700 3600 50  0001 C CNN
 F 3 "" H 1850 3650 50  0001 C CNN
@@
 P 1850 4650
 F 0 "C57" V 1598 4650 50  0000 C CNN
-F 1 "100nF" V 1689 4650 50  0000 C CNN
+F 1 "100 nF" V 1689 4650 50  0000 C CNN
 F 2 "Capacitor_SMD:C_0402_1005Metric" V 1700 4600 50  0001 C CNN
 F 3 "" H 1850 4650 50  0001 C CNN
@@
 P 1850 5700
 F 0 "C58" V 1598 5700 50  0000 C CNN
-F 1 "100nF" V 1689 5700 50  0000 C CNN
+F 1 "100 nF" V 1689 5700 50  0000 C CNN
 F 2 "Capacitor_SMD:C_0402_1005Metric" V 1700 5650 50  0001 C CNN
 F 3 "" H 1850 5700 50  0001 C CNN
@@
 P 1850 6800
 F 0 "C59" V 1598 6800 50  0000 C CNN
-F 1 "100nF" V 1689 6800 50  0000 C CNN
+F 1 "100 nF" V 1689 6800 50  0000 C CNN
 F 2 "Capacitor_SMD:C_0402_1005Metric" V 1700 6750 50  0001 C CNN
 F 3 "" H 1850 6800 50  0001 C CNN
@@
 P 1050 3300
 F 0 "C64" V 798 3300 50  0000 C CNN
-F 1 "100nF" V 889 3300 50  0000 C CNN
+F 1 "100 nF" V 889 3300 50  0000 C CNN
 F 2 "Capacitor_SMD:C_0402_1005Metric" V 900 3250 50  0001 C CNN
 F 3 "" H 1050 3300 50  0001 C CNN
