File: kicad/iobus.sch (KiCad schematic (older format))
At the start: 62 parts, among them J15 HEADER-1x02, J17 Conn_01x40_Male, J7 USBMINI, P1 HEADER_2x5, U12 MCP3424, U13 MCP3424, U14 MCP3424, U15 MCP3424, U16 MCP23017-E_SO, U17 LM2596S-5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

Commit message: a msg
Parts:
- C34, C40, C42, C44, C62, C63: value 100uF -> 100 nF
- C35, C41, C43, C46: value 10uF -> 10 uF
- C49: value 680 uF -> 680 µF
- C51, C52: value 220 uF -> 220 µF
- D2: footprint Diode_SMD:D_SMC-RM10_Universal_Handsoldering -> Diode_SMD:D_SMC
- R19, R21, R23, R25, R27, R29, R31, R33, R35, R36, R37, R41, R43, R45, R47, R49, R51, R53, R55: value 10k -> 10 k
- R20, R22, R24, R26, R28, R30, R32, R34, R42, R44, R46, R48, R50, R52, R54, R56: value 6.8k -> 6,8 k

Commit message: a msg
Parts:
- J7: footprint Connector_USB:USB_Micro-B_Molex-105133-0001 -> Connector_USB:USB_Micro-B_Wuerth_614105150721_Vertical
Changed lines of the file:
@@
 F 0 "J7" H 8382 2455 60  0000 R CNN
 F 1 "USBMINI" H 8700 2100 60  0001 C CNN
-F 2 "Connector_USB:USB_Micro-B_Molex-105133-0001" H 8686 2791 60  0001 C CNN
+F 2 "Connector_USB:USB_Micro-B_Wuerth_614105150721_Vertical" H 8686 2791 60  0001 C CNN
 F 3 "" H 8750 2450 60  0000 C CNN
 	1    8750 2450
