File: kicad/ass_shield.kicad_pcb (KiCad board)
At the start: 2 copper layers, 100 x 86 mm, 210 parts, among them J1 Conn_01x03_Male, J10 HEADER_1x4, J11 HEADER-1x08, J12 U.FL, J13 RJ11-6PTH, J14 U.FL, J15 HEADER-1x02, J16 Conn_01x03_Male, J17 Conn_01x40_Male, J18 Conn_01x38_Male, J19 HEADER-1x02-connectors, J2 DEBUG, J20 HEADER_1x4, J3 Conn_01x03_Male, J4 USB, J5 U.FL, J6 USB, J7 USBMINI, J8 U.FL, J9 RJ45, M1 CR1220SMD, P1 HEADER_2x5, Q1 BSN20, Q2 BC107, SW1 SW_DIP-8-SMT-HALFSIZE, SW2 SW_DIP-8-SMT-HALFSIZE, U1 OrangePiPC, U10 MCP2515-EST, U11 MCP2551-I-SN, U12 MCP3424, U13 MCP3424, U14 MCP3424, U15 MCP3424, U16 MCP23017-E_SO, U17 LM2596S-5, U18 LM1117-3.3, U19 CP2102-GMR_NRND, U2 DS3231M, U20 PCA9685, U21 MCP4728, U22 MCP4728, U23 MCP4728, U24 MCP4728, U3 SN65HVD72, U4 NRF24L01p, U5 RFM95HW, U6 CC2530F, U7 DS2482, U8 DS9503, U9 RFM69HW, Y1 9,84375 MHz, Y2 13,5600 MHz, Y3 4,8970 MHz, Y4 6,7458 MHz, Y5 32 MHz, Y6 16 MHz, Y7 16 MHz

Commit message: a msg
Parts:
- C10, C9: value 0,047 µF -> 47 nF
- C17, C21: value 22pF -> 22 pF
- C22, C33: value 560pF -> 560 pF
- C32, C53, C57, C58, C59, C60, C61, C64: value 100nF -> 100 nF
- C34, C40, C42, C44, C62, C63: value 100uF -> 100 nF
- C35, C41, C43, C46: value 10uF -> 10 uF
- C49: value 680 uF -> 680 µF
- C51, C52: value 220 uF -> 220 µF
- D2: footprint Diode_SMD:D_SMC-RM10_Universal_Handsoldering -> Diode_SMD:D_SMC
- J13: footprint imm:6p6c -> imm:rj11-shield
- J9: footprint w_conn_pc:rj45-shield -> imm:rj45-shield
- R1: value 100 -> 100 R
- R10, R11: value 100R -> 100 R
- R14, R19, R2, R21, R23, R25, R27, R29, R3, R31, R33, R35, R36, R37, R38, R39, R40, R41, R43, R45, R47, R49, R5, R51, R53, R55, R57, R58, R59, R7: value 10k -> 10 k
- R15, R16: value 10R -> 10 R
- R17, R18: value 120R -> 120 R
- R20, R22, R24, R26, R28, R30, R32, R34, R42, R44, R46, R48, R50, R52, R54, R56: value 6.8k -> 6,8 k
- R4: value 0 -> 0 R
- R6: value 22k -> 22 k
- R9: value 4.7k -> 4,7 k
- moved J13 1.11 mm to (153.3, 131.2)
Routing:
- net Net-(D2-Pad1): track 45.6 -> 48.5 mm
- net 5V: track 691.7 -> 690.1 mm
- net Net-(J13-Pad3): track 28.0 -> 26.8 mm

Commit message: a msg
Parts:
- added C65: 10 uF 6.3V, Capacitor_SMD:C_1206_3216Metric, F.Cu at (136.0, 93.6)
- added C66: 10 uF 6.3V, Capacitor_SMD:C_1206_3216Metric, F.Cu at (165.1, 128.0)
- added C67: 10 uF 6.3V, Capacitor_SMD:C_1206_3216Metric, F.Cu at (177.2, 89.4)
- added C68: 10 uF 6.3V, Capacitor_SMD:C_1206_3216Metric, F.Cu at (163.0, 101.8)
- added C69: 10 uF 6.3V, Capacitor_SMD:C_1206_3216Metric, F.Cu at (150.5, 84.2)
- J7: footprint Connector_USB:USB_Micro-B_Molex-105133-0001 -> Connector_USB:USB_Micro-B_Wuerth_614105150721_Vertical
- moved C9 2.41 mm to (146.7, 82.9)
- moved C32 1.16 mm to (168.5, 126.9)
- moved R2 1.16 mm to (161.9, 123.5)
- moved R3 1.16 mm to (161.9, 125.6)
- moved U7 1.16 mm to (166.3, 123.5)
- moved J7 1.11 mm to (151.3, 59.9)
Connections:
- D8 pad 3: 5V -> 3,3V
- D9 pad 3: 5V -> 3,3V
- J7 pad 4: (no net) -> Net-(J7-Pad4)
- L5 pad 1: GND -> 3,3V
- L6 pad 1: GND -> 3,3V
Routing:
- net 3,3V: track 255.0 -> 297.0 mm, vias 19 -> 21
- net 5V: track 690.1 -> 656.4 mm
- net Net-(J7-Pad2): track 4.46 -> 8.26 mm, vias 2 -> 1
- net R950: track 94.0 -> 92.0 mm
- net R69N: track 34.9 -> 33.4 mm
- net Net-(J7-Pad3): track 3.20 -> 4.27 mm
- net Net-(C63-Pad1): track 11.3 -> 10.4 mm, vias 2 -> 1
- net R95N: track 60.9 -> 60.0 mm
- net Net-(C9-Pad1): track 1.87 -> 2.67 mm
- net GND: track 26.7 -> 26.6 mm, vias 82 -> 86

Commit message: a msg
Parts:
- L5: footprint Inductor_SMD:L_0402_1005Metric -> Inductor_SMD:L_0603_1608Metric
- L6: footprint Inductor_SMD:L_0402_1005Metric -> Inductor_SMD:L_0805_2012Metric
- moved L6 0.41 mm to (138.8, 105.1)
- moved L5 0.40 mm to (138.8, 91.1)
Connections:
- J7 pad 4: Net-(J7-Pad4) -> (no net)
Routing:
- net 3,3V: track 297.0 -> 293.0 mm
- net R95N: track 60.0 -> 61.2 mm
- net R950: track 92.0 -> 93.2 mm
- net R69N: track 33.4 -> 34.6 mm
