File: kicad/ass_shield.sch (KiCad schematic (older format))
At the start: 130 parts, among them J1 Conn_01x03_Male, J10 HEADER_1x4, J11 HEADER-1x08, J12 U.FL, J13 RJ11-6PTH, J14 U.FL, J16 Conn_01x03_Male, J19 HEADER-1x02-connectors, J2 DEBUG, J20 HEADER_1x4, J3 Conn_01x03_Male, J4 USB, J5 U.FL, J6 USB, J8 U.FL, J9 RJ45, M1 CR1220SMD, Q1 BSN20, Q2 BC107, SW1 SW_DIP-8-SMT-HALFSIZE, U1 OrangePiPC, U10 MCP2515-EST, U11 MCP2551-I-SN, U2 DS3231M, U3 SN65HVD72, U4 NRF24L01p, U5 RFM95HW, U6 CC2530F, U7 DS2482, U8 DS9503, U9 RFM69HW, Y1 9,84375 MHz, Y2 13,5600 MHz, Y3 4,8970 MHz, Y4 6,7458 MHz, Y5 32 MHz, Y6 16 MHz, Y7 16 MHz

Commit message: a msg
Parts:
- C10, C9: value 0,047 µF -> 47 nF
- C17, C21: value 22pF -> 22 pF
- C22, C33: value 560pF -> 560 pF
- C32, C60, C61: value 100nF -> 100 nF
- J13: footprint imm:6p6c -> imm:rj11-shield
- J9: footprint w_conn_pc:rj45-shield -> imm:rj45-shield
- R1: value 100 -> 100 R
- R10, R11: value 100R -> 100 R
- R14, R2, R3, R5, R7: value 10k -> 10 k
- R15, R16: value 10R -> 10 R
- R17, R18: value 120R -> 120 R
- R4: value 0 -> 0 R
- R6: value 22k -> 22 k
- R9: value 4.7k -> 4,7 k
- U10: symbol Interface_CAN_LIN:MCP2515-EST -> ass_shield-rescue:MCP2515-EST-Interface_CAN_LIN
Changed lines of the file:
@@
 EESchema Schematic File Version 4
 LIBS:ass_shield-cache
-EELAYER 26 0
+EELAYER 29 0
 EELAYER END
 $Descr A4 11693 8268
@@
 P 1800 5500
 F 0 "C9" H 1915 5546 50  0000 L CNN
-F 1 "0,047 µF" H 1915 5455 50  0000 L CNN
+F 1 "47 nF" H 1915 5455 50  0000 L CNN
 F 2 "Capacitor_SMD:C_0402_1005Metric" V 1650 5450 50  0001 C CNN
 F 3 "" H 1800 5500 50  0001 C CNN
@@
 P 1800 6950
 F 0 "C10" H 1915 6996 50  0000 L CNN
-F 1 "0,047 µF" H 1915 6905 50  0000 L CNN
+F 1 "47 nF" H 1915 6905 50  0000 L CNN
 F 2 "Capacitor_SMD:C_0402_1005Metric" V 1650 6900 50  0001 C CNN
 F 3 "" H 1800 6950 50  0001 C CNN
@@
 F 0 "J9" V 4887 2044 60  0000 C CNN
 F 1 "RJ45" V 4781 2044 60  0000 C CNN
-F 2 "w_conn_pc:rj45-shield" H 4728 1938 60  0001 L CNN
+F 2 "imm:rj45-shield" H 4728 1938 60  0001 L CNN
 F 3 "" H 4300 2050 60  0000 C CNN
 	1    4300 2050
@@
 P 6950 2950
 F 0 "R1" V 6743 2950 50  0000 C CNN
-F 1 "100" V 6834 2950 50  0000 C CNN
+F 1 "100 R" V 6834 2950 50  0000 C CNN
 F 2 "Resistor_SMD:R_0402_1005Metric" V 6850 3000 50  0001 C CNN
 F 3 "" H 6950 3050 50  0001 C CNN
@@
 P 7300 2650
 F 0 "C32" V 7048 2650 50  0000 C CNN
-F 1 "100nF" V 7139 2650 50  0000 C CNN
+F 1 "100 nF" V 7139 2650 50  0000 C CNN
 F 2 "Capacitor_SMD:C_0402_1005Metric" V 7150 2600 50  0001 C CNN
 F 3 "" H 7300 2650 50  0001 C CNN
@@
 P 8400 3100
 F 0 "R2" H 8330 3054 50  0000 R CNN
-F 1 "10k" H 8330 3145 50  0000 R CNN
+F 1 "10 k" H 8330 3145 50  0000 R CNN
 F 2 "Resistor_SMD:R_0402_1005Metric" V 8300 3150 50  0001 C CNN
 F 3 "" H 8400 3200 50  0001 C CNN
@@
 P 8700 3000
 F 0 "R3" H 8630 2954 50  0000 R CNN
-F 1 "10k" H 8630 3045 50  0000 R CNN
+F 1 "10 k" H 8630 3045 50  0000 R CNN
 F 2 "Resistor_SMD:R_0402_1005Metric" V 8600 3050 50  0001 C CNN
 F 3 "" H 8700 3100 50  0001 C CNN
@@
 F 0 "J13" H 9672 2854 50  0000 R CNN
 F 1 "RJ11-6PTH" H 9672 2945 50  0000 R CNN
-F 2 "imm:6p6c" H 9930 3000 20  0001 C CNN
+F 2 "imm:rj11-shield" H 9930 3000 20  0001 C CNN
 F 3 "" H 9900 2850 60  0000 C CNN
 	1    9900 2850
@@
 P 7600 5800
 F 0 "R14" H 7670 5846 50  0000 L CNN
-F 1 "10k" H 7670 5755 50  0000 L CNN
+F 1 "10 k" H 7670 5755 50  0000 L CNN
 F 2 "Resistor_SMD:R_0402_1005Metric" V 7500 5850 50  0001 C CNN
 F 3 "" H 7600 5900 50  0001 C CNN
@@
 P 7150 6350
 F 0 "R5" V 6943 6350 50  0000 C CNN
-F 1 "10k" V 7034 6350 50  0000 C CNN
+F 1 "10 k" V 7034 6350 50  0000 C CNN
 F 2 "Resistor_SMD:R_0402_1005Metric" V 7050 6400 50  0001 C CNN
 F 3 "" H 7150 6450 50  0001 C CNN
@@
 P 7150 6000
 F 0 "R4" V 6943 6000 50  0000 C CNN
-F 1 "0" V 7034 6000 50  0000 C CNN
+F 1 "0 R" V 7034 6000 50  0000 C CNN
 F 2 "Resistor_SMD:R_0402_1005Metric" V 7050 6050 50  0001 C CNN
 F 3 "" H 7150 6100 50  0001 C CNN
@@
 P 9150 6200
 F 0 "R16" V 8943 6200 50  0000 C CNN
-F 1 "10R" V 9034 6200 50  0000 C CNN
+F 1 "10 R" V 9034 6200 50  0000 C CNN
 F 2 "Resistor_SMD:R_0402_1005Metric" V 9050 6250 50  0001 C CNN
 F 3 "" H 9150 6300 50  0001 C CNN
@@
 P 9150 5700
 F 0 "R15" V 8943 5700 50  0000 C CNN
-F 1 "10R" V 9034 5700 50  0000 C CNN
+F 1 "10 R" V 9034 5700 50  0000 C CNN
 F 2 "Resistor_SMD:R_0402_1005Metric" V 9050 5750 50  0001 C CNN
 F 3 "" H 9150 5800 50  0001 C CNN
@@
 P 10500 5950
 F 0 "R17" H 10430 5904 50  0000 R CNN
-F 1 "120R" H 10430 5995 50  0000 R CNN
+F 1 "120 R" H 10430 5995 50  0000 R CNN
 F 2 "Resistor_SMD:R_0402_1005Metric" V 10400 6000 50  0001 C CNN
 F 3 "" H 10500 6050 50  0001 C CNN
@@
 R690
 $Comp
-L Interface_CAN_LIN:MCP2515-EST U10
+L ass_shield-rescue:MCP2515-EST-Interface_CAN_LIN U10
 U 1 1 5BDB4545
 P 5800 4550
@@
 P 6650 3950
 F 0 "R7" V 6443 3950 50  0000 C CNN
-F 1 "10k" V 6534 3950 50  0000 C CNN
+F 1 "10 k" V 6534 3950 50  0000 C CNN
 F 2 "Resistor_SMD:R_0402_1005Metric" V 6550 4000 50  0001 C CNN
 F 3 "" H 6650 4050 50  0001 C CNN
@@
 P 6500 4250
 F 0 "R6" H 6430 4204 50  0000 R CNN
-F 1 "22k" H 6430 4295 50  0000 R CNN
+F 1 "22 k" H 6430 4295 50  0000 R CNN
 F 2 "Resistor_SMD:R_0402_1005Metric" V 6400 4300 50  0001 C CNN
 F 3 "" H 6500 4350 50  0001 C CNN
@@
 P 6850 4750
 F 0 "R9" H 6780 4704 50  0000 R CNN
-F 1 "4.7k" H 6780 4795 50  0000 R CNN
+F 1 "4,7 k" H 6780 4795 50  0000 R CNN
 F 2 "Resistor_SMD:R_0402_1005Metric" V 6750 4800 50  0001 C CNN
 F 3 "" H 6850 4850 50  0001 C CNN
@@
 P 5000 4650
 F 0 "C17" V 4748 4650 50  0000 C CNN
-F 1 "22pF" V 4839 4650 50  0000 C CNN
+F 1 "22 pF" V 4839 4650 50  0000 C CNN
 F 2 "Capacitor_SMD:C_0402_1005Metric" V 4850 4600 50  0001 C CNN
 F 3 "" H 5000 4650 50  0001 C CNN
@@
 P 5000 5050
 F 0 "C21" V 4748 5050 50  0000 C CNN
-F 1 "22pF" V 4839 5050 50  0000 C CNN
+F 1 "22 pF" V 4839 5050 50  0000 C CNN
 F 2 "Capacitor_SMD:C_0402_1005Metric" V 4850 5000 50  0001 C CNN
 F 3 "" H 5000 5050 50  0001 C CNN
@@
 P 8050 4550
 F 0 "R10" H 7980 4504 50  0000 R CNN
-F 1 "100R" H 7980 4595 50  0000 R CNN
+F 1 "100 R" H 7980 4595 50  0000 R CNN
 F 2 "Resistor_SMD:R_0402_1005Metric" V 7950 4600 50  0001 C CNN
 F 3 "" H 8050 4650 50  0001 C CNN
@@
 P 8550 4550
 F 0 "R11" H 8480 4504 50  0000 R CNN
-F 1 "100R" H 8480 4595 50  0000 R CNN
+F 1 "100 R" H 8480 4595 50  0000 R CNN
 F 2 "Resistor_SMD:R_0402_1005Metric" V 8450 4600 50  0001 C CNN
 F 3 "" H 8550 4650 50  0001 C CNN
@@
 P 8050 4850
 F 0 "C22" H 7935 4804 50  0000 R CNN
-F 1 "560pF" H 7935 4895 50  0000 R CNN
+F 1 "560 pF" H 7935 4895 50  0000 R CNN
 F 2 "Capacitor_SMD:C_0402_1005Metric" V 7900 4800 50  0001 C CNN
 F 3 "" H 8050 4850 50  0001 C CNN
@@
 P 8550 4850
 F 0 "C33" H 8435 4804 50  0000 R CNN
-F 1 "560pF" H 8435 4895 50  0000 R CNN
+F 1 "560 pF" H 8435 4895 50  0000 R CNN
 F 2 "Capacitor_SMD:C_0402_1005Metric" V 8400 4800 50  0001 C CNN
 F 3 "" H 8550 4850 50  0001 C CNN
@@
 P 9000 4550
 F 0 "R18" H 8930 4504 50  0000 R CNN
-F 1 "120R" H 8930 4595 50  0000 R CNN
+F 1 "120 R" H 8930 4595 50  0000 R CNN
 F 2 "Resistor_SMD:R_0402_1005Metric" V 8900 4600 50  0001 C CNN
 F 3 "" H 9000 4650 50  0001 C CNN
@@
 P 5600 3450
 F 0 "C60" V 5348 3450 50  0000 C CNN
-F 1 "100nF" V 5439 3450 50  0000 C CNN
+F 1 "100 nF" V 5439 3450 50  0000 C CNN
 F 2 "Capacitor_SMD:C_0402_1005Metric" V 5450 3400 50  0001 C CNN
 F 3 "" H 5600 3450 50  0001 C CNN
@@
 P 8600 5450
 F 0 "C61" V 8348 5450 50  0000 C CNN
-F 1 "100nF" V 8439 5450 50  0000 C CNN
+F 1 "100 nF" V 8439 5450 50  0000 C CNN
 F 2 "Capacitor_SMD:C_0402_1005Metric" V 8450 5400 50  0001 C CNN
 F 3 "" H 8600 5450 50  0001 C CNN

Commit message: a msg
Parts:
- added C65, C66, C67, C68, C69: 10 uF 6.3V, Capacitor_SMD:C_1206_3216Metric, symbol Device:CP
Connections:
- net 3,3V: now also D8.3 (VDD), D9.3 (VDD), L5.1, L6.1, C65.1, C67.1, C68.1
- net 5V: now also C66.1, C69.1; no longer D8.3 (VDD), D9.3 (VDD)
- net GND: now also C65.2, C66.2, C67.2, C68.2, C69.2; no longer L5.1, L6.1
Changed lines of the file:
@@
 Wire Wire Line
 	950  7300 850  7300
-Wire Wire Line
-	850  7650 1250 7650
 $Comp
 L power:GND #PWR07
 U 1 1 5B6F2C84
-P 1250 7650
-F 0 "#PWR07" H 1250 7400 50  0001 C CNN
-F 1 "GND" H 1255 7477 50  0001 C CNN
-F 2 "" H 1250 7650 50  0001 C CNN
-F 3 "" H 1250 7650 50  0001 C CNN
-	1    1250 7650
-	1    0    0    -1
-$EndComp
-Connection ~ 1250 7650
+P 850 7650
+F 0 "#PWR07" H 850 7400 50  0001 C CNN
+F 1 "GND" H 855 7477 50  0001 C CNN
+F 2 "" H 850 7650 50  0001 C CNN
+F 3 "" H 850 7650 50  0001 C CNN
+	1    850  7650
+	1    0    0    -1
+$EndComp
 Wire Wire Line
 	850  7300 850  7350
@@
 Wire Wire Line
 	950  5850 850  5850
-Wire Wire Line
-	850  6200 1250 6200
 $Comp
 L power:GND #PWR06
 U 1 1 5B6E4663
-P 1250 6200
-F 0 "#PWR06" H 1250 5950 50  0001 C CNN
-F 1 "GND" H 1255 6027 50  0001 C CNN
-F 2 "" H 1250 6200 50  0001 C CNN
-F 3 "" H 1250 6200 50  0001 C CNN
-	1    1250 6200
-	1    0    0    -1
-$EndComp
-Connection ~ 1250 6200
+P 850 6200
+F 0 "#PWR06" H 850 5950 50  0001 C CNN
+F 1 "GND" H 855 6027 50  0001 C CNN
+F 2 "" H 850 6200 50  0001 C CNN
+F 3 "" H 850 6200 50  0001 C CNN
+	1    850  6200
+	1    0    0    -1
+$EndComp
 Wire Wire Line
 	850  5850 850  5900
@@
 	0    1    1    0
 $EndComp
-Text GLabel 1950 5250 0    50   Input ~ 0
+Text GLabel 1800 5250 0    50   Input ~ 0
 5V
 $Comp
@@
 Connection ~ 600  5150
 Text GLabel 1850 6050 0    50   Input ~ 0
-5V
+3,3V
 Wire Wire Line
 	1650 5950 1650 6100
 Text GLabel 1850 7500 0    50   Input ~ 0
-5V
+3,3V
 Wire Wire Line
 	1650 7400 1650 7600
@@
 	8950 2950 8950 3250
 Wire Wire Line
-	8950 3250 8700 3250
+	8950 3250 8850 3250
 Wire Wire Line
 	7150 3250 7150 3050
@@
 Text GLabel 4150 3400 0    50   Input ~ 0
 5V
+Wire Wire Line
+	1850 6050 1850 6300
+Wire Wire Line
+	1850 6300 1250 6300
+Wire Wire Line
+	1250 6300 1250 6200
+Wire Wire Line
+	1850 7500 1850 7750
+Wire Wire Line
+	1850 7750 1250 7750
+Wire Wire Line
+	1250 7750 1250 7650
+$Comp
+L Device:CP C65
+U 1 1 5C49501B
+P 2000 6300
+F 0 "C65" V 2255 6300 50  0000 C CNN
+F 1 "10 uF 6.3V" V 2164 6300 50  0000 C CNN
+F 2 "Capacitor_SMD:C_1206_3216Metric" H 2038 6150 50  0001 C CNN
+F 3 "~" H 2000 6300 50  0001 C CNN
+	1    2000 6300
+	0    -1   -1   0
+$EndComp
+Connection ~ 1850 6300
+Wire Wire Line
+	2150 6300 3250 6300
+Wire Wire Line
+	3250 6300 3250 6400
+Wire Wire Line
+	3250 6400 3800 6400
+Wire Wire Line
+	3800 6400 3800 6250
+Wire Wire Line
+	3800 6250 3650 6250
+$Comp
+L Device:CP C67
+U 1 1 5C4B8DFC
+P 5000 5750
+F 0 "C67" V 5255 5750 50  0000 C CNN
+F 1 "10 uF 6.3V" V 5164 5750 50  0000 C CNN
+F 2 "Capacitor_SMD:C_1206_3216Metric" H 5038 5600 50  0001 C CNN
+F 3 "~" H 5000 5750 50  0001 C CNN
+	1    5000 5750
+	0    -1   -1   0
+$EndComp
+Wire Wire Line
+	4800 5900 4800 5750
+Wire Wire Line
+	4800 5750 4850 5750
+Connection ~ 4800 5900
+Wire Wire Line
+	5150 5750 5650 5750
+Wire Wire Line
+	5650 5750 5650 6050
+$Comp
+L Device:CP C68
+U 1 1 5C4FF872
+P 6000 700
+F 0 "C68" V 5745 700 50  0000 C CNN
+F 1 "10 uF 6.3V" V 5836 700 50  0000 C CNN
+F 2 "Capacitor_SMD:C_1206_3216Metric" H 6038 550 50  0001 C CNN
+F 3 "~" H 6000 700 50  0001 C CNN
+	1    6000 700
+	0    1    1    0
+$EndComp
+Wire Wire Line
+	6150 700  6600 700
+Wire Wire Line
+	6600 700  6600 850
+Connection ~ 6600 850
+Wire Wire Line
+	5850 700  5200 700
+Wire Wire Line
+	5200 700  5200 2150
+Wire Wire Line
+	5200 2150 5300 2150
+Connection ~ 5300 2150
+$Comp
+L Device:CP C69
+U 1 1 5C549D38
+P 7600 2650
+F 0 "C69" V 7855 2650 50  0000 C CNN
+F 1 "10 uF 6.3V" V 7764 2650 50  0000 C CNN
+F 2 "Capacitor_SMD:C_1206_3216Metric" H 7638 2500 50  0001 C CNN
+F 3 "~" H 7600 2650 50  0001 C CNN
+	1    7600 2650
+	0    -1   -1   0
+$EndComp
+Wire Wire Line
+	7750 2650 8850 2650
+Wire Wire Line
+	8850 2650 8850 3250
+Connection ~ 8850 3250
+Wire Wire Line
+	8850 3250 8700 3250
+$Comp
+L Device:CP C66
+U 1 1 5C570B15
+P 2600 5650
+F 0 "C66" V 2855 5650 50  0000 C CNN
+F 1 "10 uF 6.3V" V 2764 5650 50  0000 C CNN
+F 2 "Capacitor_SMD:C_1206_3216Metric" H 2638 5500 50  0001 C CNN
+F 3 "~" H 2600 5650 50  0001 C CNN
+	1    2600 5650
+	0    -1   -1   0
+$EndComp
+Wire Wire Line
+	2750 5650 3100 5650
+Wire Wire Line
+	3100 5650 3100 5450
+Connection ~ 3100 5450
+Wire Wire Line
+	1800 5250 1900 5250
+Wire Wire Line
+	1900 5250 1900 5650
+Wire Wire Line
+	1900 5650 2450 5650
+Connection ~ 1900 5250
+Wire Wire Line
+	1900 5250 1950 5250
 $EndSCHEMATC

Commit message: a msg
Parts:
- L5: footprint Inductor_SMD:L_0402_1005Metric -> Inductor_SMD:L_0603_1608Metric
- L6: footprint Inductor_SMD:L_0402_1005Metric -> Inductor_SMD:L_0805_2012Metric
Changed lines of the file:
@@
 F 0 "L6" V 1590 7650 50  0000 C CNN
 F 1 "820 nH" V 1499 7650 50  0000 C CNN
-F 2 "Inductor_SMD:L_0402_1005Metric" V 1250 7500 50  0001 C CNN
+F 2 "Inductor_SMD:L_0805_2012Metric" V 1250 7500 50  0001 C CNN
 F 3 "" H 1350 7650 50  0001 C CNN
 	1    1400 7650
@@
 F 0 "L5" V 1590 6200 50  0000 C CNN
 F 1 "470 nH" V 1499 6200 50  0000 C CNN
-F 2 "Inductor_SMD:L_0402_1005Metric" V 1250 6050 50  0001 C CNN
+F 2 "Inductor_SMD:L_0603_1608Metric" V 1250 6050 50  0001 C CNN
 F 3 "" H 1350 6200 50  0001 C CNN
 	1    1400 6200
